Commit message: Ernesto URDF change

File: kortex_description/arms/gen3_lite/6dof/urdf/GEN3-LITE_Mod.urdf (robot description, URDF)
Before this commit: robot KR7108-URDF, 8 links, 7 joints
Links:
- link ARM: geometry collision mesh filename=package://6dof/meshes/arm_link.STL; visual mesh filename=package://6dof/meshes/arm_link.STL
- link BASE: geometry collision mesh filename=package://6dof/meshes/base_link.STL; visual mesh filename=package://6dof/meshes/base_link.STL
- link FOREARM: geometry collision mesh filename=package://6dof/meshes/forearm_link.STL; visual mesh filename=package://6dof/meshes/forearm_link.STL
- link LOWER_WRIST: geometry collision mesh filename=package://6dof/meshes/lower_wrist_link.STL; visual mesh filename=package://6dof/meshes/lower_wrist_link.STL
- link SHOULDER: geometry collision mesh filename=package://6dof/meshes/shoulder_link.STL; visual mesh filename=package://6dof/meshes/shoulder_link.STL
- link UPPER_WRIST: geometry collision mesh filename=package://6dof/meshes/upper_wrist_link.STL; visual mesh filename=package://6dof/meshes/upper_wrist_link.STL
